Commit message: add optical frames and fix some frames

File: includes/x500_tf_publisher/x500_urdf.urdf (robot description, URDF)
Before this commit: robot x500_depth, 7 links, 6 joints
Links:
- added link camera_rgb_optical_frame
- added link depth_camera_optical_frame
Joints:
- added joint camera_rgb_optical_joint: type fixed, parent camera_rgb_frame, child camera_rgb_optical_frame, origin xyz=0 0 0 rpy=-1.57 0 -1.57
- added joint depth_camera_optical_joint: type fixed, parent depth_camera_frame, child depth_camera_optical_frame, origin xyz=0 0 0 rpy=-1.5707 0 -1.57
- added joint stereo_left_camera_optical_joint: type fixed, parent stereo_left_camera_frame, child stereo_left_camera_optical_frame, origin xyz=0 0 0 rpy=-1.5707 0 -1.57
- added joint stereo_right_camera_optical_joint: type fixed, parent stereo_right_camera_frame, child stereo_right_camera_optical_frame, origin xyz=0 0 0 rpy=-1.5707 0 -1.57
- joint camera_joint: origin xyz=.12 .03 .242 rpy=0 0 0 -> xyz=0.12 0.03 0.242 rpy=0 0.3 0
- joint camera_rgb_joint: origin xyz=0.01233 -0.03 .01878 rpy=0 0.3 0 -> xyz=0.01233 -0.03 .01878 rpy=0 0 0
- joint depth_camera_joint: origin xyz=0.01233 -0.03 .01878 rpy=0 0.3 0 -> xyz=0.01233 -0.03 .01878 rpy=0 0 0
- joint imu_joint: origin xyz=0.01233 -0.03 .014 rpy=0 0.3 0 -> xyz=0.01233 -0.03 .01878 rpy=1.57 3.14 1.57
- joint stereo_left_camera_joint: origin xyz=0.1233 0.05 0.013 rpy=0 0.3 0 -> xyz=0.1233 0.05 0.013 rpy=0 0 0
- joint stereo_right_camera_joint: origin xyz=0.1233 -0.05 0.013 rpy=0 0.3 0 -> xyz=0.1233 -0.05 0.013 rpy=0 0 0

Commit message: fix link name of left camera and pose of stereos

File: includes/x500_tf_publisher/x500_urdf.urdf (robot description, URDF)
Before this commit: robot x500_depth, 9 links, 10 joints
Links:
- added link stereo_left_camera_optical_frame
- added link stereo_right_camera_optical_frame
Joints:
- joint stereo_left_camera_joint: origin xyz=0.1233 0.05 0.013 rpy=0 0 0 -> xyz=0.01233 0.05 0.013 rpy=0 0 0
- joint stereo_right_camera_joint: origin xyz=0.1233 -0.05 0.013 rpy=0 0 0 -> xyz=0.01233 -0.05 0.013 rpy=0 0 0
