Commit message: update urdf

File: includes/gz/x500_tf_publisher/x500_urdf.urdf (robot description, URDF)
Before this commit: robot x500_depth, 11 links, 10 joints
Links:
- removed link oakd_lite_base_link
- added link OakD-Lite/base_link, mass 0.061; collision box size=0.0175 0.091 0.028; visual mesh filename=package://OakD-Lite/meshes/OakDLite.dae scale=1 1 1
Joints:
- joint camera_joint: child oakd_lite_base_link -> OakD-Lite/base_link
- joint camera_rgb_joint: parent oakd_lite_base_link -> OakD-Lite/base_link
- joint depth_camera_joint: parent oakd_lite_base_link -> OakD-Lite/base_link
- joint imu_joint: parent oakd_lite_base_link -> OakD-Lite/base_link
- joint stereo_left_camera_joint: parent oakd_lite_base_link -> OakD-Lite/base_link
- joint stereo_right_camera_joint: parent oakd_lite_base_link -> OakD-Lite/base_link

Commit message: chnage orientations

File: includes/gz/x500_tf_publisher/x500_urdf.urdf (robot description, URDF)
Before this commit: robot x500_depth, 11 links, 10 joints
Joints:
- joint camera_joint: origin xyz=0.12 0.03 0.242 rpy=0 0.3 0 -> xyz=0.12 0.03 0.242 rpy=-1.85 0.0 0
