Commit message: sim: model OAK-D S2 and align stereo vision with RTAB-Map
Generate the camera SDF and URDF from one geometry module so Gazebo,
TF, and camera_info share the S2 baseline, intrinsics, and mount.
Bridge the camera IMU, correct right-camera Tx, and add health and
accuracy checks.

File: includes/gz/x500_tf_publisher/x500_urdf.urdf (robot description, URDF)
Before this commit: robot x500_depth, 11 links, 10 joints
Links:
- removed link OakD-Lite/base_link
- removed link depth_camera_frame
- removed link depth_camera_optical_frame
- added link camera_link, mass 0.091; collision box size=0.0229 0.097 0.0295; visual box size=0.0229 0.097 0.0295
Joints:
- removed joint camera_rgb_optical_joint
- removed joint depth_camera_joint
- removed joint depth_camera_optical_joint
- removed joint stereo_left_camera_optical_joint
- removed joint stereo_right_camera_optical_joint
- added joint camera_rgb_optical_frame_joint: type fixed, parent camera_rgb_frame, child camera_rgb_optical_frame, origin xyz=0 0 0 rpy=-1.57079633 0.00000000 -1.57079633
- added joint stereo_left_camera_optical_frame_joint: type fixed, parent stereo_left_camera_frame, child stereo_left_camera_optical_frame, origin xyz=0 0 0 rpy=-1.57079633 0.00000000 -1.57079633
- added joint stereo_right_camera_optical_frame_joint: type fixed, parent stereo_right_camera_frame, child stereo_right_camera_optical_frame, origin xyz=0 0 0 rpy=-1.57079633 0.00000000 -1.57079633
- joint camera_joint: child OakD-Lite/base_link -> camera_link; origin xyz=0.12 0.03 0.242 rpy=-1.85 0.0 0 -> xyz=0.120000 0.030000 0.242000 rpy=0.000000 0.296706 0.000000
- joint camera_rgb_joint: origin xyz=0.01233 -0.03 .01878 rpy=0 0 0 -> xyz=0.011450 0.000000 0.000000 rpy=0.000000 0.000000 0.000000; parent OakD-Lite/base_link -> camera_link
- joint imu_joint: origin xyz=0.01233 -0.03 .01878 rpy=1.57 3.14 1.57 -> xyz=0.000000 0.000000 0.000000 rpy=0.000000 0.000000 0.000000; parent OakD-Lite/base_link -> camera_link
- joint stereo_left_camera_joint: origin xyz=0.01233 0.05 0.013 rpy=0 0 0 -> xyz=0.011450 0.037500 0.000000 rpy=0.000000 0.000000 0.000000; parent OakD-Lite/base_link -> camera_link
- joint stereo_right_camera_joint: origin xyz=0.01233 -0.05 0.013 rpy=0 0 0 -> xyz=0.011450 -0.037500 0.000000 rpy=0.000000 0.000000 0.000000; parent OakD-Lite/base_link -> camera_link

Commit message: sim: select oak or px4 as the IMU source
IMU_SOURCE=oak keeps the Gazebo camera IMU on /imu. IMU_SOURCE=px4
relays sensor_combined and vehicle_attitude into the same topic in
base_link, converted from FRD/NED to FLU/ENU. Camera static TFs are
parsed from the x500_depth and Oak-D SDFs so each frame has one parent.

File: includes/gz/x500_tf_publisher/x500_urdf.urdf (robot description, URDF)
Before this commit: robot x500_depth, 11 links, 10 joints
Links:
- removed link OakD-Lite/base_link
- removed link camera_rgb_frame
- removed link camera_rgb_optical_frame
- removed link depth_camera_frame
- removed link depth_camera_optical_frame
- removed link imu_link
- removed link stereo_left_camera_frame
- removed link stereo_left_camera_optical_frame
- removed link stereo_right_camera_frame
- removed link stereo_right_camera_optical_frame
Joints:
- removed joint camera_joint
- removed joint camera_rgb_joint
- removed joint camera_rgb_optical_joint
- removed joint depth_camera_joint
- removed joint depth_camera_optical_joint
- removed joint imu_joint
- removed joint stereo_left_camera_joint
- removed joint stereo_left_camera_optical_joint
- removed joint stereo_right_camera_joint
- removed joint stereo_right_camera_optical_joint

Commit message: sim: restore the base camera urdf

File: includes/gz/x500_tf_publisher/x500_urdf.urdf (robot description, URDF)
Before this commit: robot x500_depth, 1 links, 0 joints
Links:
- added link OakD-Lite/base_link, mass 0.061; collision box size=0.0175 0.091 0.028; visual mesh filename=package://OakD-Lite/meshes/OakDLite.dae scale=1 1 1
- added link camera_rgb_frame
- added link camera_rgb_optical_frame
- added link depth_camera_frame
- added link depth_camera_optical_frame
- added link imu_link
- added link stereo_left_camera_frame
- added link stereo_left_camera_optical_frame
- added link stereo_right_camera_frame
- added link stereo_right_camera_optical_frame
Joints:
- added joint camera_joint: type fixed, parent base_link, child OakD-Lite/base_link, origin xyz=0.12 0.03 0.242 rpy=-1.85 0.0 0
- added joint camera_rgb_joint: type fixed, parent OakD-Lite/base_link, child camera_rgb_frame, origin xyz=0.01233 -0.03 .01878 rpy=0 0 0
- added joint camera_rgb_optical_joint: type fixed, parent camera_rgb_frame, child camera_rgb_optical_frame, origin xyz=0 0 0 rpy=-1.57 0 -1.57
- added joint depth_camera_joint: type fixed, parent OakD-Lite/base_link, child depth_camera_frame, origin xyz=0.01233 -0.03 .01878 rpy=0 0 0
- added joint depth_camera_optical_joint: type fixed, parent depth_camera_frame, child depth_camera_optical_frame, origin xyz=0 0 0 rpy=-1.5707 0 -1.57
- added joint imu_joint: type fixed, parent OakD-Lite/base_link, child imu_link, origin xyz=0.01233 -0.03 .01878 rpy=1.57 3.14 1.57
- added joint stereo_left_camera_joint: type fixed, parent OakD-Lite/base_link, child stereo_left_camera_frame, origin xyz=0.01233 0.05 0.013 rpy=0 0 0
- added joint stereo_left_camera_optical_joint: type fixed, parent stereo_left_camera_frame, child stereo_left_camera_optical_frame, origin xyz=0 0 0 rpy=-1.5707 0 -1.57
- added joint stereo_right_camera_joint: type fixed, parent OakD-Lite/base_link, child stereo_right_camera_frame, origin xyz=0.01233 -0.05 0.013 rpy=0 0 0
- added joint stereo_right_camera_optical_joint: type fixed, parent stereo_right_camera_frame, child stereo_right_camera_optical_frame, origin xyz=0 0 0 rpy=-1.5707 0 -1.57
